Commit message: feat: add simulated lidar pipeline

File: src/robot_description/urdf/diffbot.urdf.xacro (robot description, xacro)
@@ -32,4 +32,67 @@
     </inertial>
   </link>
+  <!-- 2D LiDAR mounted on top of the chassis -->
+  <link name="lidar_link">
+    <visual>
+      <geometry>
+        <cylinder radius="0.04" length="0.04"/>
+      </geometry>
+      <material name="dark_gray">
+        <color rgba="0.15 0.15 0.15 1.0"/>
+      </material>
+    </visual>
+    <collision>
+      <geometry>
+        <cylinder radius="0.04" length="0.04"/>
+      </geometry>
+    </collision>
+    <inertial>
+      <mass value="0.1"/>
+      <inertia
+        ixx="0.0000533" ixy="0.0" ixz="0.0"
+        iyy="0.0000533" iyz="0.0"
+        izz="0.0000800"/>
+    </inertial>
+  </link>
+  <joint name="lidar_joint" type="fixed">
+    <parent link="base_link"/>
+    <child link="lidar_link"/>
+    <origin xyz="0.10 0 0.10"/>
+  </joint>
+  <!-- Gazebo 2D LiDAR sensor -->
+  <gazebo reference="lidar_link">
+    <sensor name="gpu_lidar" type="gpu_lidar">
+      <topic>/scan</topic>
+      <update_rate>10</update_rate>
+      <always_on>true</always_on>
+      <visualize>true</visualize>
+      <lidar>
+        <scan>
+          <horizontal>
+            <samples>360</samples>
+            <resolution>1</resolution>
+            <min_angle>-3.14159</min_angle>
+            <max_angle>3.14159</max_angle>
+          </horizontal>
+          <vertical>
+            <samples>1</samples>
+            <resolution>1</resolution>
+            <min_angle>0.0</min_angle>
+            <max_angle>0.0</max_angle>
+          </vertical>
+        </scan>
+        <range>
+          <min>0.12</min>
+          <max>12.0</max>
+          <resolution>0.01</resolution>
+        </range>
+        <noise>
+          <type>gaussian</type>
+          <mean>0.0</mean>
+          <stddev>0.01</stddev>
+        </noise>
+      </lidar>
+    </sensor>
+  </gazebo>
   <!-- Differential-drive wheels -->
   <xacro:macro name="drive_wheel" params="side y_offset">

Commit message: feat: add simulated imu pipeline

File: src/robot_description/urdf/diffbot.urdf.xacro (robot description, xacro)
@@ -93,4 +93,41 @@
         </noise>
       </lidar>
+    </sensor>
+  </gazebo>
+  <!-- IMU mounted near the chassis center -->
+  <link name="imu_link">
+    <visual>
+      <geometry>
+        <box size="0.04 0.03 0.015"/>
+      </geometry>
+      <material name="orange">
+        <color rgba="1.0 0.4 0.0 1.0"/>
+      </material>
+    </visual>
+    <collision>
+      <geometry>
+        <box size="0.04 0.03 0.015"/>
+      </geometry>
+    </collision>
+    <inertial>
+      <mass value="0.02"/>
+      <inertia
+        ixx="0.000001875" ixy="0.0" ixz="0.0"
+        iyy="0.000003042" iyz="0.0"
+        izz="0.000004167"/>
+    </inertial>
+  </link>
+  <joint name="imu_joint" type="fixed">
+    <parent link="base_link"/>
+    <child link="imu_link"/>
+    <origin xyz="0 0 0.065"/>
+  </joint>
+  <!-- Gazebo IMU sensor -->
+  <gazebo reference="imu_link">
+    <sensor name="imu_sensor" type="imu">
+      <topic>/imu</topic>
+      <update_rate>100</update_rate>
+      <always_on>true</always_on>
+      <visualize>false</visualize>
     </sensor>
   </gazebo>

Commit message: feat: integrate M8 fake MCU runtime

File: src/robot_description/urdf/diffbot.urdf.xacro (robot description, xacro)
@@ -2,4 +2,5 @@
 <robot xmlns:xacro="http://www.ros.org/wiki/xacro"
        name="intern_diffbot">
+  <xacro:arg name="use_fake_mcu" default="false"/>
   <material name="blue">
     <color rgba="0.10 0.30 0.80 1.0"/>
@@ -194,33 +195,65 @@
     <origin xyz="-0.15 0 -0.10"/>
   </joint>
-  <!-- Simulated hardware interface -->
-  <ros2_control name="GazeboSimSystem" type="system">
-    <hardware>
-      <plugin>gz_ros2_control/GazeboSimSystem</plugin>
-    </hardware>
-    <joint name="left_wheel_joint">
-      <command_interface name="velocity">
-        <param name="min">-10.0</param>
-        <param name="max">10.0</param>
-      </command_interface>
-      <state_interface name="position"/>
-      <state_interface name="velocity"/>
-    </joint>
-    <joint name="right_wheel_joint">
-      <command_interface name="velocity">
-        <param name="min">-10.0</param>
-        <param name="max">10.0</param>
-      </command_interface>
-      <state_interface name="position"/>
-      <state_interface name="velocity"/>
-    </joint>
-  </ros2_control>
-  <!-- Load ros2_control inside Gazebo -->
-  <gazebo>
-    <plugin
-      filename="gz_ros2_control-system"
-      name="gz_ros2_control::GazeboSimROS2ControlPlugin">
-            <parameters>$(env HOME)/robot_ws/src/diffbot_controllers.yaml</parameters>
-    </plugin>
-  </gazebo>
+  <!-- Gazebo owns the joints only in the existing physics-simulation path. -->
+  <xacro:unless value="$(arg use_fake_mcu)">
+    <ros2_control name="GazeboSimSystem" type="system">
+      <hardware>
+        <plugin>gz_ros2_control/GazeboSimSystem</plugin>
+      </hardware>
+      <joint name="left_wheel_joint">
+        <command_interface name="velocity">
+          <param name="min">-10.0</param>
+          <param name="max">10.0</param>
+        </command_interface>
+        <state_interface name="position"/>
+        <state_interface name="velocity"/>
+      </joint>
+      <joint name="right_wheel_joint">
+        <command_interface name="velocity">
+          <param name="min">-10.0</param>
+          <param name="max">10.0</param>
+        </command_interface>
+        <state_interface name="position"/>
+        <state_interface name="velocity"/>
+      </joint>
+    </ros2_control>
+    <gazebo>
+      <plugin
+        filename="gz_ros2_control-system"
+        name="gz_ros2_control::GazeboSimROS2ControlPlugin">
+              <parameters>$(env HOME)/robot_ws/src/diffbot_controllers.yaml</parameters>
+      </plugin>
+    </gazebo>
+  </xacro:unless>
+  <!-- Standalone M8 path: no Gazebo control plugin may bypass this boundary. -->
+  <xacro:if value="$(arg use_fake_mcu)">
+    <ros2_control name="DiffbotMcuSystem" type="system">
+      <hardware>
+        <plugin>diffbot_hardware/DiffbotSystemHardware</plugin>
+        <param name="left_wheel_name">left_wheel_joint</param>
+        <param name="right_wheel_name">right_wheel_joint</param>
+        <param name="encoder_counts_per_revolution">2048</param>
+        <param name="command_validity_ms">100</param>
+        <param name="state_timeout_ms">200</param>
+        <param name="activation_timeout_ms">500</param>
+        <param name="mcu_state_topic">/mcu/state</param>
+      </hardware>
+      <joint name="left_wheel_joint">
+        <command_interface name="velocity">
+          <param name="min">-10.0</param>
+          <param name="max">10.0</param>
+        </command_interface>
+        <state_interface name="position"/>
+        <state_interface name="velocity"/>
+      </joint>
+      <joint name="right_wheel_joint">
+        <command_interface name="velocity">
+          <param name="min">-10.0</param>
+          <param name="max">10.0</param>
+        </command_interface>
+        <state_interface name="position"/>
+        <state_interface name="velocity"/>
+      </joint>
+    </ros2_control>
+  </xacro:if>
 </robot>
